File: DoorLockShield.sch (EAGLE design)
At the start: 1 part

Commit message: added schematic
Parts:
- added 24V: (no value), con-ptr500:AK500/2
- added C1: (no value), rcl:CPOL-EUE7.5-16
- added FREI, L_V_T_N: (no value), con-phoenix-254:MPT4
- added IC2: 74HC595N, 74xx-eu:74HC595N
- added L_V_T_O: (no value), con-phoenix-254:MPT6
- added RANDOM: (no value), con-phoenix-254:MPT5
- added RFID: (no value), con-phoenix-254:MPT8
- added RFID-LED: (no value), con-phoenix-254:MPT3
- added R_S_D, TT: (no value), con-phoenix-254:MPT2
- added SV1: (no value), con-lstb:MA03-1
- added SV2, SV3: (no value), con-lstb:MA08-1
Connections:
- new net +5V: IC1.+5V, RANDOM-4.1
- new net 00: FREI-1.1, IC1.0
- new net 01: FREI-2.1, IC1.1
- new net 02: IC1.2, SV3.2
- new net 03: IC1.3, SV3.1
- new net 04: IC1.4
- new net 05: IC1.5, RFID-5.1
- new net 06: IC1.6
- new net 06_IN: RFID-4.1, SV1.2
- new net 07: IC1.7, IC2A.SER
- new net 08: IC1.8, IC2A.RCK
- new net 09: IC1.9, IC2A.SCK
- new net 10: IC1.10
- new net 11: IC1.11, RFID-3.1
- new net 12: IC1.12, RFID-2.1
- new net 13: IC1.13, RFID-1.1
- new net 1A: SV2.5
- new net 1B: SV2.6
- new net 24V: 24V-1.KL, SV2.1
- new net 2A: SV2.4
- new net 2B: SV2.3
- new net 3.3V: IC1.+3V3, RANDOM-3.1
- new net 5V: C1.+, IC1.+VIN, IC2A.SCL, IC2P.VCC, L_V_T_N-3.1, L_V_T_O-4.1, RFID-6.1, SV1.3, SV2.7, SV3.6
- new net A0: IC1.A0, L_V_T_O-2.1
- new net A1: IC1.A1, R_S_D-2.1
- new net A2: L_V_T_O-1.1
- new net A3: IC1.A3, TT-2.1
- new net A4: FREI-3.1, IC1.A4
- new net A5: FREI-4.1, IC1.A5
- new net AGND: C1.-, IC1.GND@1, IC1.GND@2, IC1.GND@3, IC2A.G, IC2A.QH*, IC2P.GND, L_V_T_N-4.1, L_V_T_O-5.1, L_V_T_O-6.1, RFID-7.1, RFID-8.1, R_S_D-1.1, SV2.2, SV2.8, TT-1.1
- new net AREF: IC1.AREF, RANDOM-1.1
- new net GND: 24V-2.KL, RANDOM-5.1
- new net N$1: SV1.1
- new net N$11: SV3.7
- new net N$13: SV3.5
- new net N$14: SV3.3, SV3.4
- new net N$6: IC2A.QH
- new net QA: IC2A.QA, RFID-LED-3.1
- new net QB: IC2A.QB, RFID-LED-2.1
- new net QC: IC2A.QC, RFID-LED-1.1
- new net QD: IC2A.QD, L_V_T_O-3.1
- new net QE: IC2A.QE, SV3.8
- new net QF: IC2A.QF, L_V_T_N-1.1
- new net QG: IC2A.QG, L_V_T_N-2.1
- new net RST: IC1.!RESET, RANDOM-2.1
Other:
- moved on the sheet: IC1

Commit message: finalized schematik
Parts:
- removed L_V_T_N: (no value), con-phoenix-254:MPT4
- added ETH_SD: (no value), con-phoenix-254:MPT2
- added POWER_LED, SUMMER: 1 is V & 2 is Gnd, con-phoenix-254:MPT2
- added Q1, Q2: FDN5632N-F085, FDN5632N-F085:FDN5632N-F085
- added R1, R2: 220 ohm, CommonParts:R-EU_805R0805
- RANDOM: device con-phoenix-254:MPT5 -> con-phoenix-254:MPT6
Connections:
- new net N$2: Q2.G, R1.2
- new net N$3: Q1.G, R2.2
- new net N$4: POWER_LED-2.1, Q1.D
- new net N$5: Q2.D, SUMMER-2.1
- net 04: now also ETH_SD-2.1
- net 10: now also ETH_SD-1.1
- net 5V: now also L_V_T_O-5.1, POWER_LED-1.1, SUMMER-1.1; no longer L_V_T_N-3.1
- net A2: now also IC1.A2
- net AGND: now also Q1.S, Q2.S; no longer L_V_T_N-4.1, L_V_T_O-5.1
- net GND: now also RANDOM-6.1
- net QF: now also R1.1; no longer L_V_T_N-1.1
- net QG: now also R2.1; no longer L_V_T_N-2.1
Other:
- moved on the sheet: 24V-1, 24V-2, C1, IC1, IC2, IC2P, RANDOM-1, RANDOM-2, RANDOM-3, RANDOM-4, RANDOM-5, RFID-1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

Commit message: started to add brd
Parts:
- FREI: device con-phoenix-254:MPT4 -> con-phoenix-254:MPT6
- renumbered L_V_T_O to L_TÜR, R_S_D to R_TÜR, TT to TÜR_TER.
Connections:
- removed net GND: 24V-2.KL, RANDOM-5.1, RANDOM-6.1
- new net GND24: 24V-2.KL, SV2.2
- net 5V: now also FREI-5.1
- net AGND: now also FREI-6.1, RANDOM-5.1, RANDOM-6.1; no longer SV2.2
- net N$2: now also Q1.G; no longer Q2.G
- net N$3: now also Q2.G; no longer Q1.G
- net N$4: now also Q2.D; no longer Q1.D
- net N$5: now also Q1.D; no longer Q2.D
Other:
- moved on the sheet: FREI-1, FREI-2, FREI-3, FREI-4, Q1, Q2

Commit message: added description names on sch and brd
Parts:
- added PHASEN: (no value), con-phoenix-254:MPT4
- C1: value (none) -> 470uF
Connections:
- net 02 renamed STEP
- net 03 renamed DIR
- net 04 renamed SS_SD
- net 05 renamed ROT_2_SCHWARZ_G_A
- net 07 renamed SER
- net 08 renamed RCK
- net 09 renamed SCK
- net 10 renamed ETHERNET
- net 11 renamed ROT_2_SCHWARZ_K_A
- net 12 renamed ROT_1_SCHWARZ
- net 13 renamed GRÜN_1_SCHWARZ
- net 3.3V renamed 3.3V_OUT
- net A0 renamed SCHLIESS_Z_TÜR
- net A1 renamed R_SCHALTER_TÜR
- net A2 renamed TÜR_ZU_SCHALTER
- net A3 renamed TERRASSENTÜR
- net QA renamed LED1_2_GRAUE_S
- net QB renamed LED2_1_GRAU_S
- net QC renamed LED3_GRAU
- net QD renamed RELAIS_SUMMER
- net QE renamed ENABLE
- net QF renamed SUMMER
- net QG renamed POWER_LED
- removed net 06: IC1.6
- removed net N$1: SV1.1
- removed net N$11: SV3.7
- removed net N$13: SV3.5
- removed net N$6: IC2A.QH
- new net JUMPER_SS: IC1.6, SV1.1
- new net QH: FREI-6.1, IC2A.QH
- net 1A: now also PHASEN-2.1
- net 1B: now also PHASEN-1.1
- net 2A: now also PHASEN-3.1
- net 2B: now also PHASEN-4.1
- net AGND: no longer FREI-6.1
Other:
- moved on the sheet: C1, FREI-1, FREI-2, FREI-3, FREI-4, FREI-5, FREI-6, SV2, SV3
